Commit message: we did something

File: pi/robot_workspace/src/robot_description/urdf/robot.urdf (robot description, URDF)
Before this commit: robot noonoo, 5 links, 4 joints
Joints:
- joint wheel_leftjoint: type continuous -> fixed
- joint wheel_rightjoint: type continuous -> fixed

Commit message: now we do quaternion conversion
yes, actually.

File: pi/robot_workspace/src/robot_description/urdf/robot.urdf (robot description, URDF)
Before this commit: robot noonoo, 5 links, 4 joints
Joints:
- joint laser_joint: origin xyz=0.0 0.0 0.069556 rpy=0 0 0 -> xyz=0.0 0.0 0.069556 rpy=0 0 3.1415
